File: output/pcbs/my_left.kicad_pcb (KiCad board)
At the start: 2 copper layers, 158.7 x 129.1 mm, 72 parts

Commit message: replaced nice nano pcb footprint
Parts:
- MCU1: value (none) -> nice_nano; footprint ProMicro -> nice_nano
- moved MCU1 2.81 mm to (190.4, 85.2)
Connections:
- D14 pad 2: ring_top -> inner_top
- D18 pad 2: middle_top -> inner_top
- D22 pad 2: index_top -> inner_top
- D4 pad 2: outer_num -> inner_top
- D9 pad 2: pinky_num -> inner_top
- MCU1 pad 1: VCC -> (no net)
- MCU1 pad 10: P14 -> (no net)
- MCU1 pad 11: P16 -> (no net)
- MCU1 pad 12: P10 -> (no net)
- MCU1 pad 13: P1 -> (no net)
- MCU1 pad 14: P0 -> (no net)
- MCU1 pad 15: GND -> (no net)
- MCU1 pad 16: GND -> (no net)
- MCU1 pad 17: P2 -> (no net)
- MCU1 pad 18: P3 -> (no net)
- MCU1 pad 19: P4 -> (no net)
- MCU1 pad 2: GND -> (no net)
- MCU1 pad 20: P5 -> (no net)
- MCU1 pad 21: P6 -> (no net)
- MCU1 pad 22: P7 -> (no net)
- MCU1 pad 23: P8 -> (no net)
- MCU1 pad 24: P9 -> (no net)
- MCU1 pad 3: RST -> (no net)
- MCU1 pad 4: VCC -> (no net)
- MCU1 pad 5: P21 -> (no net)
- MCU1 pad 6: P20 -> (no net)
- MCU1 pad 7: P19 -> (no net)
- MCU1 pad 8: P18 -> (no net)
- MCU1 pad 9: P15 -> (no net)
Routing:
- net inner_top: track 0.00 -> 136.1 mm

Commit message: order next week
Parts:
- removed the ? at (160.8, 141.2)
- added ?: , , F.Cu at (189.9, 61.9)
- added ?: , , F.Cu at (177.4, 80.2)
- added ?: , , F.Cu at (181.0, 105.0)
- added ?: , , F.Cu at (174.7, 68.0)
- added ?: , , F.Cu at (176.8, 94.5)
- added ?: , , F.Cu at (178.8, 99.9)
- added ?: , , F.Cu at (192.7, 106.0)
- added ?: , , F.Cu at (174.7, 85.2)
- added ?: , , F.Cu at (202.7, 99.8)
- added ?: , , F.Cu at (190.8, 103.7)
- added ?: , , F.Cu at (199.9, 104.7)
- added ?: , , F.Cu at (195.1, 62.8)
- added T1: , E73:SPDT_C128955, F.Cu at (180.3, 55.0)
- moved MH2 21.6 mm to (92.4, 46.8), turned to 2 degrees
- moved S1 4.02 mm to (64.9, 138.9), turned to 180 degrees
- moved D1 3.82 mm to (64.9, 132.9), turned to 0 degrees
- moved S6 3.68 mm to (83.9, 133.9), turned to 180 degrees
- moved D6 3.48 mm to (83.9, 127.9), turned to 0 degrees
- moved S2 3.40 mm to (64.9, 119.9), turned to 180 degrees
- moved D1 3.20 mm to (64.9, 113.9), turned to 0 degrees
- moved S7 3.03 mm to (83.9, 114.9), turned to 180 degrees
- moved D7 2.83 mm to (83.9, 108.9), turned to 0 degrees
- moved S3 2.79 mm to (64.9, 100.9), turned to 180 degrees
- moved D3 2.61 mm to (64.9, 94.9), turned to 0 degrees
- moved S8 2.39 mm to (83.9, 95.9), turned to 180 degrees
- moved S4 2.23 mm to (64.9, 81.9), turned to 180 degrees
- moved D8 2.19 mm to (83.9, 89.9), turned to 0 degrees
- moved D4 2.06 mm to (64.9, 75.9), turned to 0 degrees
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- renumbered D2 to D1
Connections:
- D1 pad 2: outer_bottom -> outer_frow
- D1 pad 2: outer_home -> inner_bottom
- D10 pad 2: pinky_frow -> inner_num
- D11 pad 2: ring_tech -> outer_frow
- D12 pad 2: ring_bottom -> inner_bottom
- D13 pad 2: ring_home -> inner_home
- D16 pad 2: middle_bottom -> inner_bottom
- D17 pad 2: middle_home -> inner_home
- D20 pad 2: index_bottom -> inner_bottom
- D21 pad 2: index_home -> inner_home
- D24 pad 2: inner_bottom -> outer_frow
- D28 pad 2: thumb_bottom -> outer_frow (x2)
- D28 pad 2: thumb_bottom -> inner_bottom
- D3 pad 2: outer_top -> inner_home
- D6 pad 2: pinky_bottom -> outer_frow
- D7 pad 2: pinky_home -> inner_bottom
- D8 pad 2: pinky_top -> inner_home
- MCU1 pad 0: (no net) -> GND
- MCU1 pad 10: (no net) -> home_default
- MCU1 pad 11: (no net) -> pinky_home
- MCU1 pad 12: (no net) -> inner_bottom
- MCU1 pad 13: (no net) -> thumb_bottom
- MCU1 pad 15: (no net) -> outer_default
- MCU1 pad 16: (no net) -> outer_frow
- MCU1 pad 18: (no net) -> pinky_frow
- MCU1 pad 20: (no net) -> pinky_top
- MCU1 pad 25: (no net) -> VCC
- MCU1 pad 5: (no net) -> inner_num
- MCU1 pad 6: (no net) -> inner_top
- MCU1 pad 7: (no net) -> inner_home
- MCU1 pad 8: (no net) -> pinky_num
- S1 pad 1: (no net) -> outer_default
- S1 pad 2: outer_bottom -> outer_default
- S10 pad 1: (no net) -> pinky_num
- S10 pad 2: pinky_frow -> pinky_num
- S11 pad 1: (no net) -> pinky_home
- S11 pad 2: ring_tech -> pinky_home
- S12 pad 1: (no net) -> pinky_home
- S12 pad 2: ring_bottom -> pinky_home
- S13 pad 1: (no net) -> pinky_home
- S13 pad 2: ring_home -> pinky_home
- S14 pad 1: (no net) -> pinky_home
- S14 pad 2: ring_top -> pinky_home
- S15 pad 1: (no net) -> pinky_home
- S15 pad 2: ring_num -> pinky_home
- S16 pad 1: (no net) -> pinky_frow
- S16 pad 2: middle_bottom -> pinky_frow
- S17 pad 1: (no net) -> pinky_frow
- S17 pad 2: middle_home -> pinky_frow
- S18 pad 1: (no net) -> pinky_frow
- S18 pad 2: middle_top -> pinky_frow
- S19 pad 1: (no net) -> pinky_frow
- S19 pad 2: middle_num -> pinky_frow
- S2 pad 1: (no net) -> outer_default
- S2 pad 2: outer_home -> outer_default
- S20 pad 1: (no net) -> pinky_top
- S20 pad 2: index_bottom -> pinky_top
- S21 pad 1: (no net) -> pinky_top
- S21 pad 2: index_home -> pinky_top
- S22 pad 1: (no net) -> pinky_top
- S22 pad 2: index_top -> pinky_top
- S23 pad 1: index_num -> pinky_top
- S23 pad 2: index_num -> pinky_top
- S24 pad 1: (no net) -> home_default
- S24 pad 2: inner_bottom -> home_default
- S25 pad 1: (no net) -> home_default
- S25 pad 2: inner_home -> home_default
- S26 pad 1: (no net) -> home_default
- S28 pad 1: (no net) -> thumb_bottom
- S29 pad 1: (no net) -> pinky_top
- S29 pad 2: outer_default -> pinky_top
- S3 pad 1: (no net) -> outer_default
- S3 pad 2: outer_top -> outer_default
- S30 pad 1: (no net) -> home_default
- S30 pad 2: near_default -> home_default
- S31 pad 1: (no net) -> thumb_bottom
- S31 pad 2: home_default -> thumb_bottom
- S4 pad 1: (no net) -> outer_default
- S4 pad 2: outer_num -> outer_default
- S5 pad 1: (no net) -> outer_default
- S5 pad 2: outer_frow -> outer_default
- S6 pad 1: (no net) -> pinky_num
- S6 pad 2: pinky_bottom -> pinky_num
- S7 pad 1: (no net) -> pinky_num
- S7 pad 2: pinky_home -> pinky_num
- S8 pad 1: (no net) -> pinky_num
- S8 pad 2: pinky_top -> pinky_num
- S9 pad 1: (no net) -> pinky_num
Routing:
- net (no net): track 79.9 -> 840.1 mm
- net outer_default: track 0.00 -> 287.9 mm, vias 0 -> 5
- net pinky_num: track 0.00 -> 265.9 mm, vias 0 -> 5
- net outer_frow: track 0.00 -> 232.0 mm
- net pinky_home: track 0.00 -> 228.4 mm, vias 0 -> 5
- net inner_bottom: track 0.00 -> 199.9 mm
- net pinky_top: track 0.00 -> 199.8 mm, vias 0 -> 5
- net pinky_frow: track 0.00 -> 190.2 mm, vias 0 -> 4
- net inner_home: track 0.00 -> 168.0 mm
- net inner_top: track 136.1 -> 204.0 mm
- net thumb_bottom: track 0.00 -> 64.6 mm, vias 0 -> 2
- net inner_num: track 155.4 -> 215.6 mm, vias 1 -> 0
- net home_default: track 100.7 -> 136.9 mm, vias 0 -> 5
- net VCC: track 18.3 -> 50.0 mm
- net RAW: track 17.2 -> 29.3 mm
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Other:
- board size 158.7 x 129.1 mm -> 156.5 x 128.9 mm

Commit message: polished pcb, generated gerber files
Parts:
- renumbered MH2 to MH1, MH2 to MH3, MH2 to MH4
Routing:
- net RAW: track 29.3 -> 28.6 mm
- net pinky_top: track 199.8 -> 199.2 mm
Other:
- rule pad_to_mask_clearance: 0.05 -> 0
